File: pcb/lightctrl.kicad_pcb (KiCad board)
At the start: 2 copper layers, 71.1 x 22.9 mm, 30 parts, among them IC1 ESP-WROOM-02, P1 LED_CONN, P2 PROG, P3 IO, P4 BATT_SENSE, P5 5V, Q1 BSS138, Q2 IRF8788, SW1 SW_FLASH, SW2 SW_RST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

Commit message: State as it is!
Parts:
- added JP3: JUMPER, solder_jumper:SOLDER_JUMPER, F.Cu at (107.6, 55.7)
- added JP4: JUMPER, solder_jumper:SOLDER_JUMPER, F.Cu at (104.6, 55.8)
- JP1, JP2: footprint Pin_Headers:Pin_Header_Straight_1x02 -> solder_jumper:SOLDER_JUMPER
- moved JP1 1.69 mm to (130.0, 55.9), turned to 0 degrees
- moved JP2 1.69 mm to (130.0, 52.1), turned to 0 degrees
Connections:
- C4 pad 1: /ESP8266/CTS -> /ESP8266/RST
- IC1 pad 15: /ESP8266/CTS -> /ESP8266/RST
- P2 pad 1: /ESP8266/BOOT_SEL -> /ESP8266/DTR
- P2 pad 2: /ESP8266/TXO -> /ESP8266/RXI
- P2 pad 3: /ESP8266/RXI -> /ESP8266/TXO
- R11 pad 1: /ESP8266/CTS -> /ESP8266/RST
- SW2 pad 2: /ESP8266/CTS -> /ESP8266/RST
- U1 pad 1: GND -> +5V
- U1 pad 2: +3V3 -> GND
- U1 pad 3: +5V -> +3V3
Routing:
- net /ESP8266/RST: track 0.00 -> 36.8 mm, vias 0 -> 2
- net /ESP8266/CTS: track 34.5 -> 9.42 mm
- net +5V: track 90.6 -> 95.6 mm, vias 3 -> 4
- net /ESP8266/TXO: track 20.2 -> 15.4 mm
- net /ESP8266/DTR: track 0.00 -> 2.77 mm
- net /ESP8266/RXI: track 18.0 -> 20.4 mm
- net +3V3: track 101.6 -> 103.2 mm
- net /ESP8266/IO12: track 62.3 -> 63.8 mm
- net GND: track 147.9 -> 149.1 mm
- net /ESP8266/BOOT_SEL: track 42.9 -> 42.1 mm
- net /ESP8266/IO13: track 57.7 -> 58.5 mm
